Commit message: add ros2 control

File: robot_2_ws/src/robot_2_description/urdf/robot_2.urdf.xacro (robot description, xacro)
@@ -1,8 +1,8 @@
 <?xml version="1.0"?>
-<robot xmlns:xacro="http://www.ros.org/wiki/xacro" name="robot_2">
-    <!-- Relative paths remain identical since files live in the same directory -->
+<robot xmlns:xacro="http://ros.org" name="robot_2">
+    <!-- Declare execution mode argument (Defaults to false for real hardware) -->
+    <xacro:arg name="sim_mode" default="false" />
     <xacro:include filename="robot_core.xacro" />
-    <xacro:include filename="gazebo_control.xacro" />
-    <!-- <xacro:include filename="ros2_control.xacro" /> -->
+    <xacro:include filename="ros2_control.xacro" />
     <xacro:include filename="lidar.xacro" />
 </robot>

File: robot_2_ws/src/robot_2_description/urdf/ros2_control.xacro (robot description, xacro)
@@ -1,35 +1,51 @@
 <?xml version="1.0"?>
 <robot xmlns:xacro="http://www.ros.org/wiki/xacro">
-  <!-- Fixed the block name to GazeboSimSystem -->
-  <ros2_control name="GazeboSimSystem" type="system">
-    <hardware>
-        <plugin>gz_ros2_control/GazeboSimSystem</plugin>
-    </hardware>
-    <!-- Cleaned up command_interfaces (Moved min/max limits to joint definitions instead) -->
-    <joint name="front_left_wheel_joint">
-      <command_interface name="velocity"/>
-      <state_interface name="position"/>
-      <state_interface name="velocity"/>
-    </joint>
-    <joint name="front_right_wheel_joint">
-      <command_interface name="velocity"/>
-      <state_interface name="position"/>
-      <state_interface name="velocity"/>
-    </joint>
-    <joint name="back_left_wheel_joint">
-      <command_interface name="velocity"/>
-      <state_interface name="position"/>
-      <state_interface name="velocity"/>
-    </joint>
-    <joint name="back_right_wheel_joint">
-      <command_interface name="velocity"/>
-      <state_interface name="position"/>
-      <state_interface name="velocity"/>
-    </joint>
-  </ros2_control>
-  <gazebo>
-    <plugin filename="gz_ros2_control-system" name="gz_ros2_control::GazeboSimSystem">
-      <parameters>$(find robot_2_bringup)/config/my_controllers.yaml</parameters>
-    </plugin>
-  </gazebo>
+  <!-- Sim Mode declared here directly inside ros2_control.xacro as per Josh Newans -->
+  <xacro:arg name="sim_mode" default="false" />
+  <!-- ========================================== -->
+  <!-- SIMULATION MODE (GAZEBO)                   -->
+  <!-- ========================================== -->
+  <xacro:if value="$(arg sim_mode)">
+    <ros2_control name="GazeboSimSystem" type="system">
+      <hardware>
+          <plugin>gz_ros2_control/GazeboSimSystem</plugin>
+      </hardware>
+      <joint name="front_left_wheel_joint"><command_interface name="velocity"/><state_interface name="position"/><state_interface name="velocity"/></joint>
+      <joint name="front_right_wheel_joint"><command_interface name="velocity"/><state_interface name="position"/><state_interface name="velocity"/></joint>
+      <joint name="back_left_wheel_joint"><command_interface name="velocity"/><state_interface name="position"/><state_interface name="velocity"/></joint>
+      <joint name="back_right_wheel_joint"><command_interface name="velocity"/><state_interface name="position"/><state_interface name="velocity"/></joint>
+    </ros2_control>
+    <gazebo>
+      <plugin filename="gz_ros2_control-system" name="gz_ros2_control::GazeboSimSystem">
+        <parameters>$(find robot_2_bringup)/config/my_controllers.yaml</parameters>
+      </plugin>
+    </gazebo>
+  </xacro:if>
+  <!-- ========================================== -->
+  <!-- REAL ROBOT HARDWARE MODE                   -->
+  <!-- ========================================== -->
+  <xacro:unless value="$(arg sim_mode)">
+    <ros2_control name="RealRobotSystem" type="system">
+      <hardware>
+        <plugin>diffdrive_arduino/DiffDriveArduinoHardware</plugin>
+        <param name="left_wheel_name">front_left_wheel_joint</param>
+        <param name="right_wheel_name">front_right_wheel_joint</param>
+        <!-- Updated to use the recommended symlink alias from your udev rules -->
+        <param name="device">/dev/ttyUSB_ARDUINO</param>
+        <param name="baud_rate">57600</param>
+        <param name="timeout_ms">2000</param>
+        <param name="enc_counts_per_rev">990</param>
+      </hardware>
+      <joint name="front_left_wheel_joint">
+        <command_interface name="velocity"/>
+        <state_interface name="position"/>
+        <state_interface name="velocity"/>
+      </joint>
+      <joint name="front_right_wheel_joint">
+        <command_interface name="velocity"/>
+        <state_interface name="position"/>
+        <state_interface name="velocity"/>
+      </joint>
+    </ros2_control>
+  </xacro:unless>
 </robot>
