Commit message: create the hardware interface

File: robot_2_ws/src/robot_2_description/urdf/ros2_control.xacro (robot description, xacro)
@@ -1,39 +1,12 @@
 <?xml version="1.0"?>
 <robot xmlns:xacro="http://www.ros.org/wiki/xacro">
-  <!-- Sim Mode declared here directly inside ros2_control.xacro as per Josh Newans -->
-  <xacro:arg name="sim_mode" default="false" />
-  <!-- ========================================== -->
-  <!-- SIMULATION MODE (GAZEBO)                   -->
-  <!-- ========================================== -->
+  <xacro:arg name="sim_mode" default="false"/>
+  <!-- ====================================================== -->
+  <!-- SIMULATION                                             -->
+  <!-- ====================================================== -->
   <xacro:if value="$(arg sim_mode)">
     <ros2_control name="GazeboSimSystem" type="system">
       <hardware>
-          <plugin>gz_ros2_control/GazeboSimSystem</plugin>
-      </hardware>
-      <joint name="front_left_wheel_joint"><command_interface name="velocity"/><state_interface name="position"/><state_interface name="velocity"/></joint>
-      <joint name="front_right_wheel_joint"><command_interface name="velocity"/><state_interface name="position"/><state_interface name="velocity"/></joint>
-      <joint name="back_left_wheel_joint"><command_interface name="velocity"/><state_interface name="position"/><state_interface name="velocity"/></joint>
-      <joint name="back_right_wheel_joint"><command_interface name="velocity"/><state_interface name="position"/><state_interface name="velocity"/></joint>
-    </ros2_control>
-    <gazebo>
-      <plugin filename="gz_ros2_control-system" name="gz_ros2_control::GazeboSimSystem">
-        <parameters>$(find robot_2_bringup)/config/my_controllers.yaml</parameters>
-      </plugin>
-    </gazebo>
-  </xacro:if>
-  <!-- ========================================== -->
-  <!-- REAL ROBOT HARDWARE MODE                   -->
-  <!-- ========================================== -->
-  <xacro:unless value="$(arg sim_mode)">
-    <ros2_control name="RealRobotSystem" type="system">
-      <hardware>
-        <plugin>diffdrive_arduino/DiffDriveArduinoHardware</plugin>
-        <param name="left_wheel_name">front_left_wheel_joint</param>
-        <param name="right_wheel_name">front_right_wheel_joint</param>
-        <!-- Updated to use the recommended symlink alias from your udev rules -->
-        <param name="device">/dev/ttyUSB_ARDUINO</param>
-        <param name="baud_rate">57600</param>
-        <param name="timeout_ms">2000</param>
-        <param name="enc_counts_per_rev">990</param>
+        <plugin>gz_ros2_control/GazeboSimSystem</plugin>
       </hardware>
       <joint name="front_left_wheel_joint">
@@ -47,4 +20,75 @@
         <state_interface name="velocity"/>
       </joint>
+      <joint name="back_left_wheel_joint">
+        <command_interface name="velocity"/>
+        <state_interface name="position"/>
+        <state_interface name="velocity"/>
+      </joint>
+      <joint name="back_right_wheel_joint">
+        <command_interface name="velocity"/>
+        <state_interface name="position"/>
+        <state_interface name="velocity"/>
+      </joint>
+    </ros2_control>
+    <gazebo>
+      <plugin
+        filename="gz_ros2_control-system"
+        name="gz_ros2_control::GazeboSimSystem">
+        <parameters>
+          $(find robot_2_bringup)/config/my_controllers.yaml
+        </parameters>
+      </plugin>
+    </gazebo>
+  </xacro:if>
+  <!-- ====================================================== -->
+  <!-- REAL ROBOT                                             -->
+  <!-- ====================================================== -->
+  <xacro:unless value="$(arg sim_mode)">
+    <ros2_control name="RealRobotSystem" type="system">
+      <hardware>
+        <plugin>robot_2_hardware/Robot2System</plugin>
+        <!-- Arduino serial configuration -->
+        <param name="device">/dev/ttyUSB_ARDUINO</param>
+        <param name="baud_rate">57600</param>
+        <param name="timeout_ms">100</param>
+        <!-- Encoder configuration -->
+        <param name="encoder_ticks_per_rev">1980</param>
+        <!-- Arduino PID period -->
+        <param name="pid_period_ms">50</param>
+        <!-- Wheel geometry -->
+        <param name="wheel_radius">0.0425</param>
+      </hardware>
+      <!-- ================================================== -->
+      <!-- LEFT FRONT                                         -->
+      <!-- ================================================== -->
+      <joint name="front_left_wheel_joint">
+        <command_interface name="velocity"/>
+        <state_interface name="position"/>
+        <state_interface name="velocity"/>
+      </joint>
+      <!-- ================================================== -->
+      <!-- LEFT REAR                                          -->
+      <!-- ================================================== -->
+      <joint name="back_left_wheel_joint">
+        <command_interface name="velocity"/>
+        <state_interface name="position"/>
+        <state_interface name="velocity"/>
+      </joint>
+      <!-- ================================================== -->
+      <!-- RIGHT FRONT                                        -->
+      <!-- ================================================== -->
+      <joint name="front_right_wheel_joint">
+        <command_interface name="velocity"/>
+        <state_interface name="position"/>
+        <state_interface name="velocity"/>
+      </joint>
+      <!-- ================================================== -->
+      <!-- RIGHT REAR                                         -->
+      <!-- ================================================== -->
+      <joint name="back_right_wheel_joint">
+        <command_interface name="velocity"/>
+        <state_interface name="position"/>
+        <state_interface name="velocity"/>
+      </joint>
     </ros2_control>
   </xacro:unless>

Commit message: refactor PID parameter and joint configuration in ros2_control.xacro

File: robot_2_ws/src/robot_2_description/urdf/ros2_control.xacro (robot description, xacro)
@@ -54,12 +54,21 @@
         <!-- Encoder configuration -->
         <param name="encoder_ticks_per_rev">1980</param>
-        <!-- Arduino PID period -->
-        <param name="pid_period_ms">50</param>
+        <!--
+          Arduino PID period, in SECONDS.
+          on_init() reads a parameter named exactly "pid_period"
+          (see getNumericParameter calls in robot_2_system.cpp),
+          NOT "pid_period_ms". 0.05s = 50ms matches config.h's
+          PID_PERIOD.
+        -->
+        <param name="pid_period">0.05</param>
         <!-- Wheel geometry -->
         <param name="wheel_radius">0.0425</param>
       </hardware>
-      <!-- ================================================== -->
-      <!-- LEFT FRONT                                         -->
-      <!-- ================================================== -->
+      <!--
+        Joint order below MUST match the index assumption hard-coded
+        in Robot2System::write()/read():
+          0 = front_left, 1 = front_right, 2 = back_left, 3 = back_right
+      -->
+      <!-- LEFT FRONT (index 0) -->
       <joint name="front_left_wheel_joint">
         <command_interface name="velocity"/>
@@ -67,7 +76,11 @@
         <state_interface name="velocity"/>
       </joint>
-      <!-- ================================================== -->
-      <!-- LEFT REAR                                          -->
-      <!-- ================================================== -->
+      <!-- RIGHT FRONT (index 1) -->
+      <joint name="front_right_wheel_joint">
+        <command_interface name="velocity"/>
+        <state_interface name="position"/>
+        <state_interface name="velocity"/>
+      </joint>
+      <!-- LEFT REAR (index 2) -->
       <joint name="back_left_wheel_joint">
         <command_interface name="velocity"/>
@@ -75,15 +88,5 @@
         <state_interface name="velocity"/>
       </joint>
-      <!-- ================================================== -->
-      <!-- RIGHT FRONT                                        -->
-      <!-- ================================================== -->
-      <joint name="front_right_wheel_joint">
-        <command_interface name="velocity"/>
-        <state_interface name="position"/>
-        <state_interface name="velocity"/>
-      </joint>
-      <!-- ================================================== -->
-      <!-- RIGHT REAR                                         -->
-      <!-- ================================================== -->
+      <!-- RIGHT REAR (index 3) -->
       <joint name="back_right_wheel_joint">
         <command_interface name="velocity"/>
